File: Dossier Janus/Projet_PAMI_Kicad.kicad_pcb (KiCad board)
At the start: 4 copper layers, 61 x 38.5 mm, 37 parts

Commit message: Rectification
Parts:
- removed AZ1117 5v: AZ1117-5.0, Package_TO_SOT_SMD:SOT-223-3_TabPin2
- removed C1: 10u, Capacitor_SMD:C_0805_2012Metric
- removed C2: 22u, Capacitor_SMD:C_0805_2012Metric
- added U12: R-78B5.0-2.0, Converter_DCDC:Converter_DCDC_RECOM_R-78B-2.0_THT, F.Cu at (125.8, 72.8)
- U7: renamed from AZ1117 3v3
- moved U6 0.59 mm to (125.0, 83.8)
- renumbered ST-LINK to J1, TP5v to TP1, TP3v3 to TP2, Servo1 to U1, Uson to U10, MCU to U11, IR to U2, Servo2 to U3, Moteur2 to U5, Moteur1 to U6, Driver to U9
Routing:
- net +5V: track 25.0 -> 8.41 mm, vias 5 -> 2
- net +7.5V: track 113.6 -> 98.8 mm
- net /SWCLK: track 13.3 -> 11.2 mm
- net /NRST: track 34.6 -> 33.7 mm
- net GND: track 0.00 -> 0.19 mm, vias 116 -> 115

Commit message: Finalisation du PCB--Dossier Janus
Parts:
- removed C15: 10u, Capacitor_SMD:C_0805_2012Metric
- removed C17: 100n, Capacitor_SMD:C_0402_1005Metric
- removed H4: MountingHole_Pad, MountingHole:MountingHole_2.7mm_M2.5_Pad
- removed J1: FTSH-107-01-F-DV-K, FTSH-107-01-F-DV-K:SAMTEC_FTSH-107-01-F-DV-K
- removed S1: 430471025826, boutonSMD_wurth430471025826:430471025826
- removed TP1, TP2: TestPoint, TestPoint:TestPoint_Pad_D2.0mm
- removed U1, U3: ~, Connector_PinHeader_2.54mm:PinHeader_1x03_P2.54mm_Vertical
- removed U10: ~, Connector_PinHeader_2.54mm:PinHeader_1x04_P2.54mm_Vertical
- removed U11: STM32L552CCTx, Package_QFP:LQFP-48_7x7mm_P0.5mm
- removed U12: R-78B5.0-2.0, Converter_DCDC:Converter_DCDC_RECOM_R-78B-2.0_THT
- removed U5, U6, U8: ~, Connector_PinHeader_2.54mm:PinHeader_1x02_P2.54mm_Vertical
- removed U7: AZ1117-3.3, Package_TO_SOT_SMD:SOT-223-3_TabPin2
- removed U9: TB6612FNG, Package_SO:SSOP-24_5.3x8.2mm_P0.65mm
- added Alim: ~, Connector_JST:JST_PH_B2B-PH-K_1x02_P2.00mm_Vertical, F.Cu at (96.9, 75.3)
- added C1: 100n, Capacitor_SMD:C_0402_1005Metric, F.Cu at (103.7, 78.8)
- added C2: 10u, Capacitor_SMD:C_0805_2012Metric, F.Cu at (131.7, 81.4)
- added Driver1: TB6612FNG, Package_SO:SSOP-24_5.3x8.2mm_P0.65mm, F.Cu at (111.3, 79.0)
- added IR1: ~, Connector_JST:JST_XH_S6B-XH-A-1_1x06_P2.50mm_Horizontal, F.Cu at (121.7, 67.9)
- added Moteur1: ~, Connector_JST:JST_XH_B2B-XH-A_1x02_P2.50mm_Vertical, B.Cu at (104.9, 95.7)
- added Moteur2: ~, Connector_JST:JST_XH_B2B-XH-A_1x02_P2.50mm_Vertical, B.Cu at (125.9, 98.2)
- added Regu5v-3v1: AZ1117-3.3, Package_TO_SOT_SMD:SOT-223-3_TabPin2, F.Cu at (132.5, 87.4)
- added Regu7v-5v1: R-78B5.0-2.0, Converter_DCDC:Converter_DCDC_RECOM_R-78B-2.0_THT, F.Cu at (96.8, 82.5)
- added ST-LINK1: FTSH-107-01-F-DV-K, FTSH-107-01-F-DV-K:SAMTEC_FTSH-107-01-F-DV-K, F.Cu at (114.9, 95.4)
- added Servo1: ~, Connector_JST:JST_PH_B3B-PH-K_1x03_P2.00mm_Vertical, F.Cu at (99.4, 68.6)
- added Servo2: ~, Connector_JST:JST_PH_B3B-PH-K_1x03_P2.00mm_Vertical, F.Cu at (108.3, 87.4)
- added Switch1: 430471025826, boutonSMD_wurth430471025826:430471025826, F.Cu at (129.2, 67.1)
- added TP-3v: TestPoint, TestPoint:TestPoint_Pad_D2.0mm, F.Cu at (122.8, 90.5)
- added TP-5v: TestPoint, TestPoint:TestPoint_Pad_D2.0mm, F.Cu at (95.8, 91.3)
- added Uson1: ~, Connector_JST:JST_PH_B4B-PH-K_1x04_P2.00mm_Vertical, F.Cu at (96.6, 61.9)
- C10: value 10n -> 100n
- C11: value 1u -> 100n
- C13: value 100n -> 1u
- C14: value 10u -> 10n; footprint Capacitor_SMD:C_0805_2012Metric -> Capacitor_SMD:C_0402_1005Metric
- C5: value 4u7 -> 100n; footprint Capacitor_SMD:C_0805_2012Metric -> Capacitor_SMD:C_0402_1005Metric
- C6: value 100n -> 10u; footprint Capacitor_SMD:C_0402_1005Metric -> Capacitor_SMD:C_0805_2012Metric
- C7: value 100n -> 4u7; footprint Capacitor_SMD:C_0402_1005Metric -> Capacitor_SMD:C_0805_2012Metric
- U2: value ~ -> MCU; footprint Connector_PinHeader_2.54mm:PinHeader_1x06_P2.54mm_Vertical -> Package_QFP:LQFP-48_7x7mm_P0.5mm
- moved G*** 74.9 mm to (92.0, 69.8)
- moved H1 47.9 mm to (92.5, 97.7)
- moved C6 43.2 mm to (104.1, 75.4), turned to 180 degrees
- moved C3 41.3 mm to (105.3, 78.5)
- moved C13 37.8 mm to (128.6, 76.6), turned to 0 degrees
- moved U2 35.8 mm to (122.2, 79.1), turned to 180 degrees
- moved C10 34.8 mm to (117.4, 82.9), turned to 180 degrees
- moved H3 32.6 mm to (138.0, 97.7)
- moved C14 32.5 mm to (134.0, 70.7), turned to 0 degrees
- moved C4 32.0 mm to (126.0, 89.4), turned to 90 degrees
- moved H2 31.7 mm to (137.0, 63.0)
- moved C12 29.8 mm to (128.5, 77.9), turned to 0 degrees
- moved C11 28.1 mm to (127.5, 83.2), turned to -90 degrees
- moved C9 27.2 mm to (118.0, 74.7), turned to 180 degrees
- moved C8 26.5 mm to (126.0, 85.0), turned to -90 degrees
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Connections:
- C10 pad 1: +3.3VA -> +3.3V
- C11 pad 1: +3.3VA -> +3.3V
- C12 pad 1: /NRST -> +3.3VA
- C13 pad 1: +7.5V -> +3.3VA
- C14 pad 1: +7.5V -> /NRST
- C3 pad 1: +5V -> +3.3V
- C5 pad 1: +3.3V -> +7.5V
- C6 pad 1: +3.3V -> +7.5V
- U2 pad 1: +5V -> +3.3V
- U2 pad 2: /IR_1 -> unconnected-(U2-PC13-Pad2)
- U2 pad 3: /IR_2 -> unconnected-(U2-PC14-Pad3)
- U2 pad 4: /IR_3 -> unconnected-(U2-PC15-Pad4)
- U2 pad 5: /IR_4 -> unconnected-(U2-PH0-Pad5)
- U2 pad 6: GND -> unconnected-(U2-PH1-Pad6)
Routing:
- net +7.5V: track 98.8 -> 22.6 mm, vias 2 -> 0
- net /STLINK_RX: track 20.3 -> 59.1 mm
- net /PWMB: track 48.1 -> 16.0 mm
- net +3.3V: track 51.5 -> 21.5 mm, vias 8 -> 19
- net /PWMA: track 38.3 -> 16.8 mm
- net /AIN1: track 31.0 -> 48.9 mm, vias 2 -> 4
- net /STLINK_TX: track 37.3 -> 21.9 mm
- net /BIN2: track 27.3 -> 42.2 mm
- net /BO1: track 44.3 -> 30.6 mm
- net /STBY: track 47.6 -> 61.1 mm, vias 2 -> 4
- net /BIN1: track 30.5 -> 42.2 mm
- net /AIN2: track 37.1 -> 48.8 mm, vias 2 -> 4
- net /Trig: track 18.5 -> 29.6 mm
- net /Echo: track 17.6 -> 28.1 mm
- net /PWM_Servo2: track 20.8 -> 11.3 mm
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- added copper zone on F.Cu, net +3.3V
- added copper zone on F.Cu, net +5V
- added copper zone on F.Cu, net +7.5V
Other:
- board size 61 x 38.5 mm -> 55 x 45.5 mm
- board text removed: "PROJET PAMI ARES 1A"

Commit message: Mise à jour couche d'alimentation
Parts:
- renumbered TP-5v to TP1, TP-3v to TP2, Alim to U1
Routing:
- net +5V: track 7.24 -> 0.00 mm, vias 14 -> 16
Changed lines of the file:
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@@
 		(descr "JST PH series connector, B2B-PH-K (http://www.jst-mfg.com/product/pdf/eng/ePH.pdf), generated with kicad-footprint-generator")
 		(tags "connector JST PH side entry")
-		(property "Reference" "Alim"
+		(property "Reference" "U1"
 			(at 1.883 -2.669 180)
 			(layer "F.SilkS")
@@
 		(descr "SMD pad as test Point, diameter 2.0mm")
 		(tags "test point SMD pad")
-		(property "Reference" "TP-5v"
+		(property "Reference" "TP1"
 			(at -0.088 2.107 0)
 			(layer "F.SilkS")
@@
 		(descr "SMD pad as test Point, diameter 2.0mm")
 		(tags "test point SMD pad")
-		(property "Reference" "TP-3v"
+		(property "Reference" "TP2"
 			(at -2.097 0.552 180)
 			(layer "F.SilkS")
@@
 		(tags "connector JST PH side entry")
 		(property "Reference" "Uson1"
-			(at -3.1 -0.5 90)
+			(at 3 -2.9 0)
 			(layer "F.SilkS")
 			(effects
@@
 			(at 3 4 0)
 			(layer "F.Fab")
-			(hide yes)
 			(effects
 				(font
@@
 		(layer "Edge.Cuts")
 	)
-	(segment
-		(start 130.749 81.407)
-		(end 130.749 83.638)
-		(width 0.3)
-		(layer "F.Cu")
-		(net 1)
-	)
-	(segment
-		(start 134.3 79.9)
-		(end 132.256 79.9)
-		(width 0.3)
-		(layer "F.Cu")
-		(net 1)
-	)
-	(segment
-		(start 132.256 79.9)
-		(end 130.749 81.407)
-		(width 0.3)
-		(layer "F.Cu")
-		(net 1)
-	)
-	(segment
-		(start 130.749 83.638)
-		(end 130.161 84.226)
-		(width 0.3)
-		(layer "F.Cu")
-		(net 1)
-	)
 	(via
 		(at 100.23 87.36)
@@
 	)
 	(via
+		(at 134.89 79.76)
+		(size 0.45)
+		(drill 0.3)
+		(layers "F.Cu" "B.Cu")
+		(free yes)
+		(net 1)
+	)
+	(via
 		(at 98.33 88.32)
 		(size 0.45)
@@
 	)
 	(via
+		(at 135.89 79.76)
+		(size 0.45)
+		(drill 0.3)
+		(layers "F.Cu" "B.Cu")
+		(free yes)
+		(net 1)
+	)
+	(via
 		(at 102.12 85.58)
 		(size 0.45)
@@
 	)
 	(via
-		(at 134.3 79.9)
+		(at 133.89 79.76)
 		(size 0.45)
 		(drill 0.3)
 		(layers "F.Cu" "B.Cu")
-		(teardrops
-			(best_length_ratio 0.5)
-			(max_length 1)
-			(best_width_ratio 1)
-			(max_width 2)
-			(curve_points 0)
-			(filter_ratio 0.9)
-			(enabled no)
-			(allow_two_segments no)
-			(prefer_zone_connections yes)
-		)
+		(free yes)
 		(net 1)
 	)
@@
 	)
 	(segment
+		(start 130.14 78.46)
+		(end 130.13 78.47)
+		(width 0.2)
+		(layer "F.Cu")
+		(net 5)
+	)
+	(segment
+		(start 130.13 78.47)
+		(end 127.50741 78.47)
+		(width 0.2)
+		(layer "F.Cu")
+		(net 5)
+	)
+	(segment
 		(start 118.50141 87.541685)
 		(end 120.343096 85.7)
@@
 	)
 	(segment
+		(start 127.50741 78.47)
+		(end 127.10641 78.871)
+		(width 0.2)
+		(layer "F.Cu")
+		(net 5)
+	)
+	(segment
 		(start 121.629 78.871)
 		(end 126.3365 78.871)
@@
 	)
 	(segment
+		(start 127.10641 78.871)
+		(end 126.3365 78.871)
+		(width 0.2)
+		(layer "F.Cu")
+		(net 5)
+	)
+	(segment
 		(start 120.343096 85.7)
 		(end 121 85.7)
@@
 		(net 5)
 	)
-	(segment
-		(start 130.35 78.55)
-		(end 130.029 78.871)
-		(width 0.2)
-		(layer "F.Cu")
-		(net 5)
-	)
-	(segment
-		(start 130.029 78.871)
-		(end 126.3365 78.871)
-		(width 0.2)
-		(layer "F.Cu")
-		(net 5)
-	)
 	(via
-		(at 130.35 78.55)
+		(at 130.14 78.46)
 		(size 0.45)
 		(drill 0.3)
@@
 	)
 	(segment
-		(start 130.35 78.55)
-		(end 130.8 78.1)
+		(start 121 79.5)
+		(end 121 85.7)
 		(width 0.2)
 		(layer "B.Cu")
@@
 	)
 	(segment
-		(start 121 79.5)
-		(end 121 85.7)
+		(start 130.8 77.8)
+		(end 130.8 72.5)
 		(width 0.2)
 		(layer "B.Cu")
@@
 	)
 	(segment
-		(start 130.8 78.1)
-		(end 130.8 72.5)
+		(start 130.8 72.5)
+		(end 131.159 72.141)
 		(width 0.2)
 		(layer "B.Cu")
@@
 	)
 	(segment
-		(start 130.8 72.5)
-		(end 131.159 72.141)
+		(start 130.14 78.46)
+		(end 130.8 77.8)
 		(width 0.2)
 		(layer "B.Cu")
@@
 	)
 	(zone
+		(net 1)
+		(net_name "+5V")
+		(layer "F.Cu")
+		(hatch edge 0.5)
+		(priority 4)
+		(connect_pads yes
+			(clearance 0.2)
+		)
+		(min_thickness 0.25)
+		(filled_areas_thickness no)
+		(fill yes
+			(thermal_gap 0.5)
+			(thermal_bridge_width 0.5)
+		)
+		(polygon
+			(pts
+				(xy 136.19 80.16) (xy 131.25 80.17) (xy 131.25 82.15) (xy 130.91 82.15) (xy 130.91 85.24) (xy 129.39 85.25)
+				(xy 129.39 83.16) (xy 130.03 83.14) (xy 130.04 79.66) (xy 130.75 79.34) (xy 136.19 79.33)
+			)
+		)
+	)
+	(zone
 		(net 2)
 		(net_name "GND")
@@
 		(polygon
 			(pts
-				(xy 125.09 57.75) (xy 125 72.5) (xy 101.6 72.4) (xy 101.6 80.1) (xy 113.72 80.1) (xy 113.73 90.63)
-				(xy 109.44 90.63) (xy 109.44 100.3) (xy 136 100.3) (xy 136 82.6) (xy 131.41 82.6) (xy 131.41 86.07)
-				(xy 128.98 86.07) (xy 128.98 79.2) (xy 133.23 79.2) (xy 133.23 57.75)
+				(xy 124.99 72.5) (xy 125 72.5) (xy 101.6 72.4) (xy 101.6 80.1) (xy 113.72 80.1) (xy 113.73 90.63)
+				(xy 109.44 90.63) (xy 109.44 100.3) (xy 136 100.3) (xy 136 82.6) (xy 133.23 82.6) (xy 133.23 82.6)
+				(xy 133.23 82.6) (xy 133.23 79.2) (xy 133.23 79.2) (xy 133.13 72.5)
 			)
 		)
