File: Dossier Janus-bis/Janus_finalV/Janus_finalV.kicad_pcb (KiCad board)
At the start: 4 copper layers, 41 x 52.4 mm, 35 parts, among them J1 Conn_01x02, J10 Conn_01x02, J2 Conn_01x04, J3 BU33SD5WG-TR, J4 R-78B5.0-2.0, J5 Conn_01x03, J6 Conn_01x03, J7 Conn_ST_STDC14, J8 Conn_01x06, J9 Conn_01x02, U1 STM32L552CCTx

Commit message: Update final Version
Parts:
- added J11: Conn_01x04, Connector_PinHeader_2.54mm:PinHeader_1x04_P2.54mm_Vertical, F.Cu at (147.7, 75.0)
- added J14: Conn_01x04, Connector_PinHeader_2.54mm:PinHeader_1x04_P2.54mm_Vertical, F.Cu at (147.7, 80.1)
- added J15: Conn_01x04, Connector_PinHeader_2.54mm:PinHeader_1x04_P2.54mm_Vertical, F.Cu at (147.7, 77.5)
- moved C11 4.61 mm to (147.4, 65.2)
- moved Switch1 3.42 mm to (144.8, 69.5), turned to 180 degrees
- moved TP2 1.99 mm to (126.1, 71.1)
Connections:
- U1 pad 18: unconnected-(U1-PB0-Pad18) -> GPIO1
- U1 pad 19: unconnected-(U1-PB1-Pad19) -> GPIO2
- U1 pad 20: unconnected-(U1-PB2-Pad20) -> GPIO3
- U1 pad 21: unconnected-(U1-PB10-Pad21) -> GPIO4
Routing:
- net GPIO1: track 0.00 -> 36.7 mm, vias 0 -> 1
- net GPIO2: track 0.00 -> 34.5 mm, vias 0 -> 1
- net GPIO4: track 0.00 -> 33.6 mm, vias 0 -> 1
- net GPIO3: track 0.00 -> 31.3 mm, vias 0 -> 1
- net +3.3V: track 21.4 -> 23.4 mm, vias 9 -> 15
- net NRST: track 22.6 -> 24.1 mm
- net PWMB: track 17.1 -> 16.1 mm
- net GND: vias 249 -> 254
- net +7.5V: vias 2 -> 5
