File: Dossier Janus-bis/Janus_finalV/Janus_finalV.kicad_sch (KiCad schematic)
At the start: 34 parts, among them J1 Conn_01x02, J10 Conn_01x02, J2 Conn_01x04, J3 BU33SD5WG-TR, J4 R-78B5.0-2.0, J5 Conn_01x03, J6 Conn_01x03, J7 Conn_ST_STDC14, J8 Conn_01x06, J9 Conn_01x02, U1 STM32L552CCTx

Commit message: Update final Version
Parts:
- added J11, J14, J15: Conn_01x04, Connector_PinHeader_2.54mm:PinHeader_1x04_P2.54mm_Vertical, symbol Connector_Generic:Conn_01x04
Connections:
- net +3.3V: now also J15.1 (Pin_1), J15.2 (Pin_2), J15.3 (Pin_3), J15.4 (Pin_4)
- net GND: now also J14.1 (Pin_1), J14.2 (Pin_2), J14.3 (Pin_3), J14.4 (Pin_4)
- net GPIO1: now reaches U1.18 (PB0)
- net GPIO1: now also J11.1 (Pin_1)
- net GPIO2: now reaches U1.19 (PB1)
- net GPIO2: now also J11.2 (Pin_2)
- net GPIO3: now reaches U1.20 (PB2)
- net GPIO3: now also J11.3 (Pin_3)
- net GPIO4: now reaches U1.21 (PB10)
- net GPIO4: now also J11.4 (Pin_4)
- no-connect marks 24 -> 20
Other:
- note added: "Pin GPIO & GND"
- moved on the sheet: C1, C2, C3, C4, C5, C6, Driver1, H1, H2, H3, H4, J1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

Commit message: update PCB1A
Changed lines of the file:
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@@
 (kicad_sch
-	(version 20231120)
+	(version 20250114)
 	(generator "eeschema")
-	(generator_version "8.0")
+	(generator_version "9.0")
 	(paper "A4")
 	(title_block
@@
 		(comment 1 "Capodagli Janus")
 	)
+	(rectangle
+		(start 189.23 124.46)
+		(end 228.6 162.56)
+		(stroke
+			(width 0)
+			(type default)
+		)
+		(fill
+			(type none)
+		)
+	)
+	(rectangle
+		(start 109.22 115.57)
+		(end 175.26 195.58)
+		(stroke
+			(width 0)
+			(type default)
+		)
+		(fill
+			(type none)
+		)
+	)
+	(rectangle
+		(start 17.78 80.01)
+		(end 55.88 114.3)
+		(stroke
+			(width 0)
+			(type default)
+		)
+		(fill
+			(type none)
+		)
+	)
+	(rectangle
+		(start 240.03 127)
+		(end 279.4 162.56)
+		(stroke
+			(width 0)
+			(type default)
+		)
+		(fill
+			(type none)
+		)
+	)
+	(rectangle
+		(start 34.29 21.59)
+		(end 59.69 66.04)
+		(stroke
+			(width 0)
+			(type default)
+		)
+		(fill
+			(type none)
+		)
+	)
+	(rectangle
+		(start 182.88 13.97)
+		(end 275.59 121.92)
+		(stroke
+			(width 0)
+			(type default)
+		)
+		(fill
+			(type none)
+		)
+	)
+	(rectangle
+		(start 130.81 13.97)
+		(end 180.34 69.85)
+		(stroke
+			(width 0)
+			(type default)
+		)
+		(fill
+			(type none)
+		)
+	)
+	(rectangle
+		(start 17.78 115.57)
+		(end 100.33 195.58)
+		(stroke
+			(width 0)
+			(type default)
+		)
+		(fill
+			(type none)
+		)
+	)
+	(rectangle
+		(start 66.04 76.2)
+		(end 127 104.14)
+		(stroke
+			(width 0)
+			(type default)
+		)
+		(fill
+			(type none)
+		)
+	)
+	(rectangle
+		(start 83.82 13.97)
+		(end 125.73 60.96)
+		(stroke
+			(width 0)
+			(type default)
+		)
+		(fill
+			(type none)
+		)
+	)
+	(text "Trous de fixation\n"
+		(exclude_from_sim no)
+		(at 46.99 24.13 0)
+		(effects
+			(font
+				(size 1.27 1.27)
+			)
+		)
+	)
+	(text "Servos"
+		(exclude_from_sim no)
+		(at 105.41 16.51 0)
+		(effects
+			(font
+				(size 1.27 1.27)
+				(thickness 0.254)
+				(bold yes)
+			)
+		)
+	)
+	(text "Moteurs\n"
+		(exclude_from_sim no)
+		(at 262.89 129.54 0)
+		(effects
+			(font
+				(size 1.27 1.27)
+				(thickness 0.254)
+				(bold yes)
+			)
+		)
+	)
+	(text "Module infra-rouge\n"
+		(exclude_from_sim no)
+		(at 207.01 129.54 0)
+		(effects
+			(font
+				(size 1.27 1.27)
+				(thickness 0.254)
+				(bold yes)
+			)
+		)
+	)
+	(text "Connecteur ST-Link\n"
+		(exclude_from_sim no)
+		(at 154.94 16.51 0)
+		(effects
+			(font
+				(size 1.27 1.27)
+				(thickness 0.254)
+				(bold yes)
+			)
+		)
+	)
+	(text "Ultra-son"
+		(exclude_from_sim no)
+		(at 35.56 85.09 0)
+		(effects
+			(font
+				(size 1.27 1.27)
+				(thickness 0.254)
+				(bold yes)
+			)
+		)
+	)
+	(text "Alimentation des piles et régulateurs de tension"
+		(exclude_from_sim no)
+		(at 60.96 119.38 0)
+		(effects
+			(font
+				(size 1.5 1.5)
+			)
+		)
+	)
+	(text "Motor Driver\n"
+		(exclude_from_sim no)
+		(at 142.24 119.38 0)
+		(effects
+			(font
+				(size 1.27 1.27)
+			)
+		)
+	)
+	(text "Pin GPIO & GND \n"
+		(exclude_from_sim no)
+		(at 99.06 78.74 0)
+		(effects
+			(font
+				(size 1.27 1.27)
+				(thickness 0.254)
+				(bold yes)
+			)
+		)
+	)
+	(text "MCU\n"
+		(exclude_from_sim no)
+		(at 232.41 16.51 0)
+		(effects
+			(font
+				(size 1.27 1.27)
+				(thickness 0.254)
+				(bold yes)
+			)
+		)
+	)
 	(junction
 		(at 243.84 30.48)
@@
 		)
 	)
-	(rectangle
-		(start 189.23 124.46)
-		(end 228.6 162.56)
-		(stroke
-			(width 0)
-			(type default)
-		)
-		(fill
-			(type none)
-		)
-	)
-	(rectangle
-		(start 109.22 115.57)
-		(end 175.26 195.58)
-		(stroke
-			(width 0)
-			(type default)
-		)
-		(fill
-			(type none)
-		)
-	)
-	(rectangle
-		(start 17.78 80.01)
-		(end 55.88 114.3)
-		(stroke
-			(width 0)
-			(type default)
-		)
-		(fill
-			(type none)
-		)
-	)
-	(rectangle
-		(start 240.03 127)
-		(end 279.4 162.56)
-		(stroke
-			(width 0)
-			(type default)
-		)
-		(fill
-			(type none)
-		)
-	)
-	(rectangle
-		(start 34.29 21.59)
-		(end 59.69 66.04)
-		(stroke
-			(width 0)
-			(type default)
-		)
-		(fill
-			(type none)
-		)
-	)
-	(rectangle
-		(start 182.88 13.97)
-		(end 275.59 121.92)
-		(stroke
-			(width 0)
-			(type default)
-		)
-		(fill
-			(type none)
-		)
-	)
-	(rectangle
-		(start 130.81 13.97)
-		(end 180.34 69.85)
-		(stroke
-			(width 0)
-			(type default)
-		)
-		(fill
-			(type none)
-		)
-	)
-	(rectangle
-		(start 17.78 115.57)
-		(end 100.33 195.58)
-		(stroke
-			(width 0)
-			(type default)
-		)
-		(fill
-			(type none)
-		)
-	)
-	(rectangle
-		(start 66.04 76.2)
-		(end 127 104.14)
-		(stroke
-			(width 0)
-			(type default)
-		)
-		(fill
-			(type none)
-		)
-	)
-	(rectangle
-		(start 83.82 13.97)
-		(end 125.73 60.96)
-		(stroke
-			(width 0)
-			(type default)
-		)
-		(fill
-			(type none)
-		)
-	)
-	(text "Trous de fixation\n"
-		(exclude_from_sim no)
-		(at 46.99 24.13 0)
-		(effects
-			(font
-				(size 1.27 1.27)
-			)
-		)
-	)
-	(text "Servos"
-		(exclude_from_sim no)
-		(at 105.41 16.51 0)
-		(effects
-			(font
-				(size 1.27 1.27)
-				(thickness 0.254)
-				(bold yes)
-			)
-		)
-	)
-	(text "Moteurs\n"
-		(exclude_from_sim no)
-		(at 262.89 129.54 0)
-		(effects
-			(font
-				(size 1.27 1.27)
-				(thickness 0.254)
-				(bold yes)
-			)
-		)
-	)
-	(text "Module infra-rouge\n"
-		(exclude_from_sim no)
-		(at 207.01 129.54 0)
-		(effects
-			(font
-				(size 1.27 1.27)
-				(thickness 0.254)
-				(bold yes)
-			)
-		)
-	)
-	(text "Connecteur ST-Link\n"
-		(exclude_from_sim no)
-		(at 154.94 16.51 0)
-		(effects
-			(font
-				(size 1.27 1.27)
-				(thickness 0.254)
-				(bold yes)
-			)
-		)
-	)
-	(text "Ultra-son"
-		(exclude_from_sim no)
-		(at 35.56 85.09 0)
-		(effects
-			(font
-				(size 1.27 1.27)
-				(thickness 0.254)
-				(bold yes)
-			)
-		)
-	)
-	(text "Alimentation des piles et régulateurs de tension"
-		(exclude_from_sim no)
-		(at 60.96 119.38 0)
-		(effects
-			(font
-				(size 1.5 1.5)
-			)
-		)
-	)
-	(text "Motor Driver\n"
-		(exclude_from_sim no)
-		(at 142.24 119.38 0)
-		(effects
-			(font
-				(size 1.27 1.27)
-			)
-		)
-	)
-	(text "Pin GPIO & GND \n"
-		(exclude_from_sim no)
-		(at 99.06 78.74 0)
-		(effects
-			(font
-				(size 1.27 1.27)
-				(thickness 0.254)
-				(bold yes)
-			)
-		)
-	)
-	(text "MCU\n"
-		(exclude_from_sim no)
-		(at 232.41 16.51 0)
-		(effects
-			(font
-				(size 1.27 1.27)
-				(thickness 0.254)
-				(bold yes)
-			)
-		)
-	)
 	(label "NRST"
 		(at 214.63 45.72 0)
@@
 		)
 	)
+	(embedded_fonts no)
 )
