File: PCB finalV/Janus_finalV.kicad_pcb (KiCad board)
At the start: 4 copper layers, 41 x 52.4 mm, 38 parts, among them J1 Conn_01x02, J10 Conn_01x02, J11 Conn_01x04, J14 Conn_01x04, J15 Conn_01x04, J2 Conn_01x04, J3 BU33SD5WG-TR, J4 R-78B5.0-2.0, J5 Conn_01x03, J6 Conn_01x03, J7 Conn_ST_STDC14, J8 Conn_01x06, J9 Conn_01x02, U1 STM32L552CCTx

Commit message: MAJ code PAMI
Parts:
- added R1: 75, Resistor_SMD:R_0402_1005Metric_Pad0.72x0.64mm_HandSolder, B.Cu at (142.6, 71.8)
- added R2: 49.9, Resistor_SMD:R_0402_1005Metric_Pad0.72x0.64mm_HandSolder, B.Cu at (141.1, 71.8)
- Switch1: footprint boutonSMD_wurth430471025826:430471025826 -> bouton_Wurth_SMD:430471025826
Connections:
- J11 pad 3: GPIO3 -> Net-(J11-Pin_3)
- J11 pad 4: GPIO4 -> Net-(J11-Pin_4)
- J8 pad 1: +5V -> +3.3V
- U1 pad 20: GPIO3 -> RedLED
- U1 pad 21: GPIO4 -> YellowLED
Routing:
- net GPIO4: track 33.6 -> 0.00 mm, vias 1 -> 0
- net GPIO3: track 31.3 -> 0.00 mm, vias 1 -> 0
- net YellowLED: track 0.00 -> 29.2 mm, vias 0 -> 1
- net RedLED: track 0.00 -> 27.5 mm, vias 0 -> 1
- net Net-(J11-Pin_4): track 0.00 -> 3.05 mm
- net GPIO2: track 34.5 -> 37.4 mm
- net Net-(J11-Pin_3): track 0.00 -> 2.61 mm
- net GPIO1: track 36.7 -> 37.4 mm
- net BO1: track 8.73 -> 8.06 mm
- net GND: vias 257 -> 271

Commit message: update_final
Other:
- board text added: "Par C.Janus"
Changed lines of the file:
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@@
 			(psa4output no)
 			(plot_black_and_white yes)
-			(plotinvisibletext no)
 			(sketchpadsonfab no)
 			(plotpadnumbers no)
@@
 		(layer "Edge.Cuts")
 	)
+	(gr_text "Par C.Janus"
+		(at 142.9 41.25 0)
+		(layer "B.SilkS")
+		(effects
+			(font
+				(size 1 1)
+				(thickness 0.1)
+			)
+			(justify left bottom mirror)
+		)
+	)
 	(via
